File: hello_my_name_is/hello_my_name_is.kicad_pcb (KiCad board)
At the start: 2 copper layers, 59 x 31.5 mm, 79 parts, among them J1 USB_C_Receptacle_USB2.0, J2 OLED, P1 SAO 2x3 IDC, Q1 AO3401A, Q2 AO3400A, SW1 SSSS811101, SW2 TS-1187A-B-A-B, SW3 TS-1187A-B-A-B, SW4 TS-1187A-B-A-B, SW5 TS-1187A-B-A-B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

Commit message: uploading gerbers, going in hot w/ no review
shotgunned this 2 layer board routing in a few hours... hot garbage!
Parts:
- C25: moved to F.Cu
- moved R19 49.2 mm to (74.1, 132.6)
- moved C28 46.5 mm to (66.9, 133.4)
- moved C20 41.9 mm to (89.0, 130.8), turned to 0 degrees
- moved U4 41.7 mm to (70.1, 129.6), turned to 180 degrees
- moved C14 40.5 mm to (84.5, 133.1), turned to -90 degrees
- moved C2 40.5 mm to (98.6, 120.3), turned to 180 degrees
- moved C12 39.7 mm to (92.6, 146.4)
- moved Y1 38.6 mm to (89.4, 128.3), turned to -90 degrees
- moved R20 38.2 mm to (78.0, 131.4)
- moved C13 37.9 mm to (80.9, 133.1), turned to -90 degrees
- moved C4 35.7 mm to (99.7, 126.2), turned to 180 degrees
- moved U1 35.3 mm to (99.2, 123.2), turned to -90 degrees
- moved C21 34.9 mm to (89.0, 125.8), turned to 180 degrees
- moved D3 34.3 mm to (92.1, 144.8)
- moved R7 34.0 mm to (92.6, 147.6)
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Connections:
- D1 pad 3: /PAGE2/GPIO21 -> /PAGE2/GPIO6
- R15 pad 2: /PAGE2/GPIO19 -> /PAGE2/GPIO1
- R16 pad 2: /PAGE2/GPIO20 -> /PAGE2/GPIO0
- SW4 pad 2: /PAGE2/GPIO19 -> /PAGE2/GPIO1
- SW5 pad 2: /PAGE2/GPIO20 -> /PAGE2/GPIO0
Routing:
- net +3V3: track 0.00 -> 213.3 mm, vias 0 -> 10
- net VBUS: track 0.00 -> 126.9 mm
- net GND: track 0.00 -> 109.9 mm, vias 0 -> 40
- net /PAGE2/I2C0_SCL: track 0.00 -> 52.8 mm, vias 0 -> 4
- net /PAGE2/I2C0_SDA: track 0.00 -> 50.7 mm, vias 0 -> 4
- net /PAGE2/GPIO1: track 0.00 -> 49.2 mm, vias 0 -> 4
- net /PAGE2/GPIO0: track 0.00 -> 43.9 mm, vias 0 -> 4
- net /PAGE2/USBBOOT: track 0.00 -> 42.5 mm
- net /PAGE2/~{RESET}: track 0.00 -> 42.1 mm, vias 0 -> 4
- net Net-(D4-Pad1): track 0.00 -> 39.3 mm, vias 0 -> 4
- net /PAGE2/GPIO22: track 0.00 -> 35.9 mm, vias 0 -> 6
- net /PAGE2/GPIO6: track 0.00 -> 32.9 mm, vias 0 -> 3
- net /PAGE2/USB_D-: track 0.00 -> 32.8 mm
- net /PAGE2/USB_D+: track 0.00 -> 31.7 mm
- net /PAGE2/WS2812_DOUT: track 0.00 -> 29.0 mm, vias 0 -> 2
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- added copper zone on F.Cu, net +3V3
- added copper zone on B.Cu, net GND
- added copper zone on F.Cu, net GND
- added copper zone on F.Cu, net Net-(C10-Pad2)
- added copper zone on F.Cu, net Net-(D3-Pad2)
- added copper zone on F.Cu, net Net-(R7-Pad2)
- added copper zone on F.Cu, net VCC
Other:
- rule pad_to_mask_clearance: 0.05 -> 0
- board text added: "JLCJLCJLCJLC"
- board text added: "MS V1.0"
