File: hello_my_name_is/page2.kicad_sch (KiCad schematic)
At the start: 51 parts

Commit message: sch push before review, some component grouping
Parts:
- added C11: 4.7u, Capacitor_SMD:C_0402_1005Metric, symbol Device:C_Small
- added C24, C25, C26, C27, C28, C5, C6, C8, C9: 1u, Capacitor_SMD:C_0402_1005Metric, symbol Device:C_Small
- added C7: 2.2u, Capacitor_SMD:C_0402_1005Metric, symbol Device:C_Small
- added FID1, FID2: Fiducial, Fiducial:Fiducial_1mm_Mask2mm, symbol Mechanical:Fiducial
- added H1, H2, H3, H4: Tooling_Hole_JLC, ftp:JLC_Tooling_Hole, symbol Mechanical:MountingHole
- added H5, H6: Tooling_Hole_JLC, MountingHole:MountingHole_3.2mm_M3, symbol Mechanical:MountingHole
- added J2: OLED, Display:OLED-128O064D, symbol Connector_Generic:Conn_01x30
- added R10: 330k, Resistor_SMD:R_0402_1005Metric, symbol Device:R_Small_US
- added R11, R12: 4.7k, Resistor_SMD:R_0402_1005Metric, symbol Device:R_Small_US
- added R14, R15, R16: 10k, Resistor_SMD:R_0402_1005Metric, symbol Device:R_Small_US
- added SW4, SW5: TS-1187A-B-A-B, Button_Switch_SMD:SW_SPST_TL3342, symbol Switch:SW_Push
- BT1: renamed from BT?; footprint (none) -> ftp:BatteryHolder_MPD_BC2AAPC_2xAA_mod-SMD
- C10: renamed from C?; value ? -> 3.3p; lcsc C52923 -> C1565
- D1, D2, D4, D5: renamed from D?; LCSC C965555 -> (none); lcsc (none) -> C965555
- F1: renamed from F?; value Fuse_Small -> 24V 500mA PTC; footprint (none) -> Fuse:Fuse_0805_2012Metric; desc (none) -> NonAsm; lcsc (none) -> C910822
- L1: renamed from L?; value 10u -> 3.3u; footprint (none) -> Inductor_SMD:L_Bourns-SRN4018; desc (none) -> ftp: Not Exact, 1.23A 3.3uH ±20% 70mΩ; lcsc (none) -> C431259
- R7: renamed from R?; value ? -> 200k; lcsc (none) -> C25764
- R8: renamed from R?; value ? -> 51k; lcsc (none) -> C25794
- R9: renamed from R?; value ? -> 150k; lcsc (none) -> C25755
- SW1: renamed from SW?; footprint (none) -> ftp:SSSS811101
- U1: renamed from U?; Field5 3V3 600mA LDO -> (none); desc (none) -> 3V3 600mA LDO; lcsc lcsc -> C841192
- U2: renamed from U?; lcsc (none) -> C7722
- U4: renamed from U?; footprint Package_SON:WSON-8-1EP_6x5mm_P1.27mm_EP3.4x4mm -> Package_SO:SOIC-8W_5.3x5.3mm_P1.27mm; lcsc (none) -> C179171
- gave numbers to parts that had none: 36
Connections:
- net i2c0_scl is gone; now on net I2C0_SCL: P1.4 (SCL)
- net i2c0_sda is gone; now on net I2C0_SDA: P1.3 (SDA)
- net sao1_gpio1 is gone; now on net GPIO22: P1.5 (GPIO1)
- net +3V3: now also C24.1, C25.1, C26.1, C27.1, C28.1, C5.1, C6.1, J2.11 (Pin_11), J2.6 (Pin_6), J2.9 (Pin_9), R11.1, R12.1, R14.1, R15.1, R16.1
- net +BATT: now also SW1.3 (C); no longer SW1.1 (A)
- net GND: now also C11.1, C24.2, C25.2, C26.2, C27.2, C28.2, C5.2, C6.2, C7.1, J2.1 (Pin_1), J2.10 (Pin_10), J2.12 (Pin_12), J2.13 (Pin_13), J2.15 (Pin_15), J2.16 (Pin_16), J2.17 (Pin_17), J2.21 (Pin_21), J2.22 (Pin_22), J2.23 (Pin_23), J2.24 (Pin_24), J2.25 (Pin_25), J2.29 (Pin_29), J2.30 (Pin_30), J2.8 (Pin_8), R10.1, SW4.1, SW5.1
- net GPIO15: now also J2.14 (Pin_14), R14.2
- net GPIO19: now also R15.2, SW4.2
- net GPIO20: now also R16.2, SW5.2
- net GPIO16 renamed I2C0_SDA
- net I2C0_SDA: now also J2.19 (Pin_19), J2.20 (Pin_20), R12.2
- net GPIO17 renamed I2C0_SCL
- net I2C0_SCL: now also J2.18 (Pin_18), R11.2
- new net: C11.2, J2.28 (Pin_28)
- new net: C8.2, J2.2 (Pin_2)
- new net: J2.26 (Pin_26), R10.2
- new net: C7.2, J2.27 (Pin_27)
- new net: C8.1, J2.3 (Pin_3)
- new net: C9.2, J2.4 (Pin_4)
- new net: C9.1, J2.5 (Pin_5)
Other:
- note added: "BS0"
- note added: "BS1"
- note added: "BS2"
- note added: "C1N"
- note added: "C1P"
- note added: "C2N"
- note added: "C2P"
- note added: "CS#"
- note added: "D/C#"
- note added: "D/CP (ADDR): 0111100b' GND 0x3C <- 0111101b' VDD 0x3D"
- note added: "D0"
- note added: "D1"
- note added: "D2"
- note added: "D3"
- note added: "D4"
- note added: "D5"
- note added: "D6"
- note added: "D7"
- note added: "DOWN"
- note added: "E/RD#"
- note added: "Fiducials"
- note added: "IREF"
- note added: "Mounting"
- note added: "N.C."
- note added: "N.C. (GND)"
- note added: "NO HV BATT SO NO LEAK CIR."
- note added: "R/W#"
- note added: "RES#"
- note added: "Tooling Holes"
- note added: "UP"
- note added: "VCC"
- note added: "VCOMH"
- note added: "VDD"
- note added: "VDDB"
- note added: "VLSS"
- note added: "VSS"
- moved on the sheet: P1, R19, U4

Commit message: uploading gerbers, going in hot w/ no review
shotgunned this 2 layer board routing in a few hours... hot garbage!
Connections:
- net GPIO0: now also R16.2, SW5.2
- net GPIO1: now also R15.2, SW4.2
- net GPIO19: no longer R15.2, SW4.2
- net GPIO20: no longer R16.2, SW5.2
- net GPIO21: no longer D1.3 (DIN)
- net GPIO6: now also D1.3 (DIN)
Changed lines of the file:
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@@
     (effects (font (size 1.27 1.27)) (justify right bottom))
   )
-  (label "GPIO21" (at 68.58 185.42 180)
-    (effects (font (size 1.27 1.27)) (justify right bottom))
+  (label "GPIO6" (at 68.58 185.42 0)
+    (effects (font (size 1.27 1.27)) (justify left bottom))
   )
   (label "~{QSPI_CS}" (at 262.89 27.94 0)
     (effects (font (size 1.27 1.27)) (justify left bottom))
+  )
+  (label "GPIO1" (at 226.06 140.335 180)
+    (effects (font (size 1.27 1.27)) (justify right bottom))
   )
   (label "GPIO0" (at 273.05 45.72 180)
@@
   (label "GPIO22" (at 55.245 168.275 0)
     (effects (font (size 1.27 1.27)) (justify left bottom))
-  )
-  (label "GPIO19" (at 226.06 140.335 180)
-    (effects (font (size 1.27 1.27)) (justify right bottom))
   )
   (label "~{RESET}" (at 207.01 72.39 0)
@@
     (effects (font (size 1.27 1.27)) (justify right bottom))
   )
-  (label "GPIO20" (at 226.06 157.48 180)
+  (label "GPIO0" (at 226.06 157.48 180)
     (effects (font (size 1.27 1.27)) (justify right bottom))
   )

Commit message: sw transfer
Parts:
- H5, H6: value Tooling_Hole_JLC -> Mounting_Hole
